File: projects/test_project/test_project.kicad_sch (KiCad schematic)
At the start: 0 parts

Commit message: modify test_project
Parts:
- added D1: GREEN, LED_THT:LED_D5.0mm, symbol Device:LED
- added J1: POWER_PIN, Connector_JST:JST_XH_B2B-XH-A_1x02_P2.50mm_Vertical, symbol Connector:Conn_01x02_Pin
- added R1: 4k7, Resistor_THT:R_Axial_DIN0411_L9.9mm_D3.6mm_P12.70mm_Horizontal, symbol Device:R
- added SW1: SW_SPST, Button_Switch_THT:SW_DIP_SPSTx01_Slide_9.78x4.72mm_W7.62mm_P2.54mm, symbol Switch:SW_SPST
Connections:
- new net: D1.2 (A), R1.2
- new net +5V: J1.1 (Pin_1), SW1.2 (B)
- new net GND: D1.1 (K), J1.2 (Pin_2)
- new net SW_5V: R1.1, SW1.1 (A)
